File: kicad/siteshift/siteshift.kicad_pcb (KiCad board)
At the start: 2 copper layers, 46 parts, among them SW1 Reset, U1 DRV8873HPWPRQ1, U2 Pico, U3 LM78M05_TO252, U4 ULN2004A

Commit message: PCB design update
Parts:
- added G***: LOGO, LOGO, F.Cu at (128.0, 112.5)
- added H3: MountingHole, MountingHole:MountingHole_3.2mm_M3, F.Cu at (135.0, 55.0)
- added H3: MountingHole, MountingHole:MountingHole_3.2mm_M3, F.Cu at (35.0, 125.0)
- added H3: MountingHole, MountingHole:MountingHole_3.2mm_M3, F.Cu at (135.0, 125.0)
- added H3: MountingHole, MountingHole:MountingHole_3.2mm_M3, F.Cu at (35.0, 55.0)
- moved R4 165.9 mm to (105.0, 115.8), turned to 90 degrees
- moved C9 154.3 mm to (102.0, 115.8), turned to 90 degrees
- moved C11 151.2 mm to (101.3, 91.8)
- moved R6 149.0 mm to (101.3, 89.2)
- moved R11 138.0 mm to (100.0, 68.5), turned to 90 degrees
- moved R10 137.5 mm to (100.0, 63.0), turned to 90 degrees
- moved D1 132.9 mm to (104.8, 73.0), turned to 90 degrees
- moved R2 123.9 mm to (67.1, 91.0)
- moved C3 120.6 mm to (70.6, 65.4), turned to 180 degrees
- moved R8 117.6 mm to (43.0, 114.0), turned to 90 degrees
- moved R9 113.5 mm to (40.5, 114.0), turned to 90 degrees
- moved R1 111.4 mm to (43.8, 98.5)
- moved R7 109.9 mm to (45.5, 114.0), turned to 90 degrees
- moved R5 104.8 mm to (43.8, 101.2)
- moved LED_SIGNAL1 95.1 mm to (42.6, 125.0), turned to 0 degrees
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- renumbered SW1 to RESET
Connections:
- U2 pad 31: RV_SPEED_F -> IPROP_F
- U2 pad 34: IPROP_F -> RV_SPEED_F
Routing:
- net AGND: track 0.00 -> 168.7 mm, vias 0 -> 2
- net SW_INVERSE: track 0.00 -> 85.7 mm, vias 0 -> 2
- net GND: track 127.7 -> 210.1 mm, vias 92 -> 82
- net +12V: track 138.8 -> 214.9 mm, vias 0 -> 3
- net SW_MODE: track 0.00 -> 71.5 mm, vias 0 -> 2
- net IPROP: track 0.00 -> 59.5 mm, vias 0 -> 3
- net SW_STATE_MAN: track 0.00 -> 55.4 mm
- net SW_STATE_SEQ: track 0.00 -> 55.4 mm
- net Net-(D1-K): track 0.00 -> 46.8 mm, vias 0 -> 1
- net D_RIGHT_PWR: track 0.00 -> 44.1 mm, vias 0 -> 1
- net SW_RIGHT: track 0.00 -> 40.9 mm
- net IPROP_F: track 0.00 -> 40.2 mm
- net MOTOR_FB_F: track 0.00 -> 39.0 mm, vias 0 -> 1
- net +3.3V: track 30.2 -> 67.3 mm, vias 0 -> 1
- net Net-(U4-O5): track 2.54 -> 35.2 mm, vias 0 -> 2
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- added copper zone on B.Cu, net (none)
- added copper zone on F.Cu, net (none)
- added copper zone on F.Cu, net +12V
Other:
- board outline added: 108.5 x 81.5 mm
- board text added: "+12V"
- board text added: "1"
- board text added: "COMMUNICATION"
- board text added: "FB"
- board text added: "FB+"
- board text added: "FB-"
- board text added: "GND"
- board text added: "M"
- board text added: "M+"
- board text added: "M-"
- board text added: "MOTOR"
- board text added: "POWER"
- board text added: "RX"
- board text added: "Rv SPEED"
- board text added: "S"
- board text added: "SCL"
- board text added: "SDA"
- board text added: "SINGAL LED"
- board text added: "SW INVERSE"
- board text added: "SW LEFT"
- board text added: "SW MODE"
- board text added: "SW RIGHT"
- board text added: "SW STATE"
- board text added: "Siteshift board v0.0.0"
- board text added: "TX"
