File: kicad/siteshift/siteshift.kicad_pcb (KiCad board)
At the start: 2 copper layers, 108.5 x 81.5 mm, 51 parts, among them U1 DRV8873HPWPRQ1, U2 Pico, U3 LM78M05_TO252, U4 ULN2004A

Commit message: Changed name
Other:
- board text added: "Sideshift board v0.0.0"
- board text removed: "Siteshift board v0.0.0"
Changed lines of the file:
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@@
 		)
 	)
-	(gr_text "Siteshift board\nv0.0.0"
+	(gr_text "Sideshift board\nv0.0.0"
 		(at 136.5 95 0)
 		(layer "F.SilkS")

Commit message: First code setup
Parts:
- renumbered RESET to SW1
Changed lines of the file:
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@@
 			(net 5 "GND")
 			(pinfunction "GND")
-			(pintype "bidirectional")
+			(pintype "power_in")
 		)
 		(pad "38" smd rect
@@
 			(net 5 "GND")
 			(pinfunction "GND")
-			(pintype "bidirectional")
+			(pintype "power_in")
 		)
 		(pad "39" thru_hole oval
@@
 		(descr "tactile push button, 6x6mm e.g. PHAP33xx series, height=5mm")
 		(tags "tact sw push 6mm")
-		(property "Reference" "RESET"
+		(property "Reference" "SW1"
 			(at 3.25 -2 90)
 			(layer "F.SilkS")
@@
 			(net 6 "DVDD")
 			(pinfunction "DVDD")
-			(pintype "power_in")
+			(pintype "power_out")
 			(solder_mask_margin 0.102)
 		)
@@
 			(net 26 "IPROP")
 			(pinfunction "IPROPI2")
-			(pintype "output")
+			(pintype "passive")
 			(solder_mask_margin 0.102)
 		)
@@
 			(net 5 "GND")
 			(pinfunction "SRC")
-			(pintype "output")
+			(pintype "passive")
 			(solder_mask_margin 0.102)
 		)
@@
 			(net 5 "GND")
 			(pinfunction "SRC")
-			(pintype "output")
+			(pintype "passive")
 			(solder_mask_margin 0.102)
 		)
@@
 			(net 1 "Net-(U1-CPH)")
 			(pinfunction "CPH")
-			(pintype "power_in")
+			(pintype "passive")
 			(solder_mask_margin 0.102)
 		)
@@
 			(net 2 "Net-(U1-CPL)")
 			(pinfunction "CPL")
-			(pintype "power_in")
+			(pintype "passive")
 			(solder_mask_margin 0.102)
 		)
@@
 			(net 5 "GND")
 			(pinfunction "GND")
-			(pintype "power_in")
+			(pintype "passive")
 			(solder_mask_margin 0.102)
 		)
